File: prj/zf-filter/zf-filter.kicad_sch (KiCad schematic)
At the start: 62 parts

Commit message: zf-filter r1.0
Other:
- title: (none) -> ZF-Filter
Changed lines of the file:
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@@
 	(generator_version "8.0")
 	(paper "A4")
+	(title_block
+		(title "ZF-Filter")
+		(date "2024-03-20")
+		(rev "1.0")
+	)
 	(junction
 		(at 175.26 78.74)

Commit message: zf-filter r0.1
Parts:
- D10, D20, D30, D40, D50, D60, D70, D80: footprint Diode_SMD:D_SOD-323 -> imports:D-THT-P6KE
- renumbered JP2 to JP10, JP4 to JP2, JP3 to JP20, JP5 to JP30, JP6 to JP40
Changed lines of the file:
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@@
 		(on_board yes)
 		(dnp no)
-		(property "Reference" "JP5"
+		(property "Reference" "JP30"
 			(at 184.404 32.258 90)
 			(effects
@@
 			(project "zf-filter"
 				(path "/cb150eac-6942-474e-becf-b9054a8e99cd"
-					(reference "JP5")
+					(reference "JP30")
 					(unit 1)
 				)
@@
 			)
 		)
-		(property "Footprint" "Diode_SMD:D_SOD-323"
+		(property "Footprint" "imports:D-THT-P6KE"
 			(at 97.79 106.68 0)
 			(effects
@@
 			)
 		)
-		(property "Footprint" "Diode_SMD:D_SOD-323"
+		(property "Footprint" "imports:D-THT-P6KE"
 			(at 128.27 106.68 0)
 			(effects
@@
 			)
 		)
-		(property "Footprint" "Diode_SMD:D_SOD-323"
+		(property "Footprint" "imports:D-THT-P6KE"
 			(at 229.87 106.68 0)
 			(effects
@@
 			)
 		)
-		(property "Footprint" "Diode_SMD:D_SOD-323"
+		(property "Footprint" "imports:D-THT-P6KE"
 			(at 199.39 106.68 0)
 			(effects
@@
 			)
 		)
-		(property "Footprint" "Diode_SMD:D_SOD-323"
+		(property "Footprint" "imports:D-THT-P6KE"
 			(at 260.35 106.68 0)
 			(effects
@@
 		(dnp no)
 		(fields_autoplaced yes)
-		(property "Reference" "JP4"
+		(property "Reference" "JP2"
 			(at 153.67 31.7499 90)
 			(effects
@@
 			(project "zf-filter"
 				(path "/cb150eac-6942-474e-becf-b9054a8e99cd"
-					(reference "JP4")
+					(reference "JP2")
 					(unit 1)
 				)
@@
 		(on_board yes)
 		(dnp no)
-		(property "Reference" "JP2"
+		(property "Reference" "JP10"
 			(at 52.324 32.004 90)
 			(effects
@@
 			(project "zf-filter"
 				(path "/cb150eac-6942-474e-becf-b9054a8e99cd"
-					(reference "JP2")
+					(reference "JP10")
 					(unit 1)
 				)
@@
 			)
 		)
-		(property "Footprint" "Diode_SMD:D_SOD-323"
+		(property "Footprint" "imports:D-THT-P6KE"
 			(at 67.31 106.68 0)
 			(effects
@@
 			)
 		)
-		(property "Footprint" "Diode_SMD:D_SOD-323"
+		(property "Footprint" "imports:D-THT-P6KE"
 			(at 168.91 106.68 0)
 			(effects
@@
 		(on_board yes)
 		(dnp no)
-		(property "Reference" "JP3"
+		(property "Reference" "JP20"
 			(at 110.998 31.75 90)
 			(effects
@@
 			(project "zf-filter"
 				(path "/cb150eac-6942-474e-becf-b9054a8e99cd"
-					(reference "JP3")
+					(reference "JP20")
 					(unit 1)
 				)
@@
 			)
 		)
-		(property "Footprint" "Diode_SMD:D_SOD-323"
+		(property "Footprint" "imports:D-THT-P6KE"
 			(at 36.83 106.68 0)
 			(effects
@@
 		(on_board yes)
 		(dnp no)
-		(property "Reference" "JP6"
+		(property "Reference" "JP40"
 			(at 243.078 32.258 90)
 			(effects
@@
 			(project "zf-filter"
 				(path "/cb150eac-6942-474e-becf-b9054a8e99cd"
-					(reference "JP6")
+					(reference "JP40")
 					(unit 1)
 				)
