File: prj/zf-filter/zf-filter.kicad_pcb (KiCad board)
At the start: 2 copper layers, 172 x 60 mm, 66 parts

Commit message: zf-filter r1.0
Parts:
- removed the REF** at (230.0, 85.0)
- removed the REF** at (70.0, 125.0)
- removed the REF** at (70.0, 85.0)
- removed the REF** at (230.0, 125.0)
- added REF**: MountingHole_3.2mm_M3, MountingHole:MountingHole_3.2mm_M3, F.Cu at (70.0, 85.0)
- added REF**: MountingHole_3.2mm_M3, MountingHole:MountingHole_3.2mm_M3, F.Cu at (150.0, 85.0)
- added REF**: MountingHole_3.2mm_M3, MountingHole:MountingHole_3.2mm_M3, F.Cu at (230.0, 85.0)
- added REF**: MountingHole_3.2mm_M3, MountingHole:MountingHole_3.2mm_M3, F.Cu at (230.0, 125.0)
- added REF**: MountingHole_3.2mm_M3, MountingHole:MountingHole_3.2mm_M3, F.Cu at (70.0, 125.0)
- added REF**: MountingHole_3.2mm_M3, MountingHole:MountingHole_3.2mm_M3, F.Cu at (150.0, 125.0)
- moved SENT4 2.70 mm to (128.3, 130.0)
- moved C51 2.50 mm to (164.8, 100.5)
- moved C52 2.50 mm to (160.0, 105.2)
- moved C61 2.50 mm to (180.8, 100.5)
- moved C62 2.50 mm to (176.0, 105.2)
- moved C71 2.50 mm to (196.8, 100.5)
- moved C72 2.50 mm to (192.0, 105.2)
- moved C81 2.50 mm to (212.8, 100.5)
- moved C82 2.50 mm to (208.0, 105.2)
- moved D50 2.50 mm to (172.5, 120.2)
- moved D60 2.50 mm to (188.2, 120.2)
- moved D70 2.50 mm to (204.2, 120.2)
- moved D80 2.50 mm to (220.2, 120.2)
- moved JP4 2.50 mm to (166.5, 81.0)
- moved R51 2.50 mm to (159.7, 114.5)
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Routing:
- net 5Va: track 176.9 -> 132.3 mm
- net S4b: track 44.0 -> 54.7 mm
- net S4a: track 43.7 -> 54.4 mm
- net Net-(C82-Pad1): track 0.00 -> 9.79 mm
- net 5Vb: track 124.9 -> 132.5 mm
- net Net-(D40-A1): track 19.3 -> 21.2 mm
- net Net-(D80-A1): track 19.4 -> 20.6 mm
- net S1b: track 35.7 -> 34.8 mm
- net S3b: track 36.6 -> 37.4 mm
- net Net-(D70-A1): track 19.3 -> 20.1 mm
- net S3a: track 36.3 -> 37.2 mm
- net Net-(D30-A1): track 19.4 -> 20.2 mm
- net GND: vias 242 -> 246
Other:
- board size 172 x 60 mm -> 179 x 60 mm
- board text added: "5V"
- board text added: "GND"
- board text added: "S1"
- board text added: "S2"
- board text added: "S3"
- board text added: "S4"
- board text added: "S5"
- board text added: "S6"
- board text added: "S7"
- board text added: "S8"
- board text removed: "${REFERENCE}"

Commit message: zf-filter r0.1
Parts:
- removed REF** (x6): MountingHole_3.2mm_M3, MountingHole:MountingHole_3.2mm_M3
- D10, D20, D30, D40, D50, D60, D70, D80: footprint Diode_SMD:D_SOD-323 -> imports:D-THT-P6KE
- moved R13 23.9 mm to (86.5, 95.9), turned to -90 degrees
- moved R42 14.2 mm to (137.5, 95.9), turned to -90 degrees
- moved R32 14.1 mm to (122.5, 95.9), turned to -90 degrees
- moved R12 14.1 mm to (92.5, 95.9), turned to -90 degrees
- moved R22 14.1 mm to (107.5, 95.9), turned to -90 degrees
- moved C12 14.0 mm to (95.8, 106.1), turned to 90 degrees
- moved R23 13.8 mm to (101.5, 106.1), turned to 90 degrees
- moved R33 13.5 mm to (116.5, 106.1), turned to 90 degrees
- moved R43 13.3 mm to (131.5, 106.1), turned to 90 degrees
- moved C22 13.0 mm to (110.8, 106.1), turned to 90 degrees
- moved C32 12.2 mm to (125.8, 106.1), turned to 90 degrees
- moved R11 11.6 mm to (89.5, 106.1), turned to 90 degrees
- moved D40 11.5 mm to (131.5, 115.6), turned to 90 degrees
- moved C42 11.2 mm to (140.8, 106.1), turned to 90 degrees
- moved R21 11.0 mm to (104.5, 106.1), turned to 90 degrees
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- renumbered JP2 to JP10, JP4 to JP2, JP3 to JP20, JP5 to JP30, JP6 to JP40
Connections:
- net S1a renamed S10
- net S1b renamed S50
- net S2a renamed S20
- net S2b renamed S60
- net S3a renamed S30
- net S3b renamed S70
- net S4a renamed S40
- net S4b renamed S80
Routing:
- net Net-(D10-A1): track 19.4 -> 57.1 mm
- net Net-(D20-A1): track 20.0 -> 57.1 mm
- net Net-(D30-A1): track 20.2 -> 57.2 mm
- net Net-(D40-A1): track 21.2 -> 54.3 mm
- net 5Va: track 132.3 -> 163.2 mm
- net S40: track 54.4 -> 34.0 mm
- net S10: track 34.8 -> 14.4 mm
- net S20: track 32.6 -> 13.8 mm
- net S30: track 37.2 -> 23.8 mm
- net Net-(C12-Pad1): track 9.50 -> 6.25 mm
- net Net-(C32-Pad1): track 9.28 -> 6.08 mm
- net Net-(C22-Pad1): track 9.39 -> 6.25 mm
- net Net-(C42-Pad1): track 9.28 -> 6.26 mm
- net Net-(D50-A1): track 19.6 -> 17.0 mm
- net Net-(D80-A1): track 20.6 -> 18.3 mm
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Other:
- board size 179 x 60 mm -> 150 x 55 mm

Commit message: Add SamacSys loader libs
Parts:
- added REF**: MountingHole_3.2mm_M3, MountingHole:MountingHole_3.2mm_M3, F.Cu at (80.0, 85.0)
- added REF**: MountingHole_3.2mm_M3, MountingHole:MountingHole_3.2mm_M3, F.Cu at (220.0, 85.0)
- added REF**: MountingHole_3.2mm_M3, MountingHole:MountingHole_3.2mm_M3, F.Cu at (150.0, 130.0)
- added REF**: MountingHole_3.2mm_M3, MountingHole:MountingHole_3.2mm_M3, F.Cu at (150.0, 85.0)
- added REF**: MountingHole_3.2mm_M3, MountingHole:MountingHole_3.2mm_M3, F.Cu at (220.0, 130.0)
- added REF**: MountingHole_3.2mm_M3, MountingHole:MountingHole_3.2mm_M3, F.Cu at (80.0, 130.0)
- moved R53 26.9 mm to (156.5, 95.9), turned to -90 degrees
- moved D80 19.4 mm to (201.5, 115.6)
- moved D70 18.4 mm to (186.5, 115.6)
- moved R82 17.5 mm to (207.5, 95.9), turned to -90 degrees
- moved D60 17.4 mm to (171.5, 115.6)
- moved R72 16.9 mm to (192.5, 95.9), turned to -90 degrees
- moved D50 16.4 mm to (156.5, 115.6)
- moved R62 16.4 mm to (177.5, 95.9), turned to -90 degrees
- moved R52 15.9 mm to (162.5, 95.9), turned to -90 degrees
- moved R83 14.5 mm to (201.5, 106.1), turned to 90 degrees
- moved R73 14.1 mm to (186.5, 106.1), turned to 90 degrees
- moved R63 13.8 mm to (171.5, 106.1), turned to 90 degrees
- moved C81 9.22 mm to (207.5, 92.9)
- moved R81 9.00 mm to (204.5, 106.1), turned to 90 degrees
- moved R71 8.70 mm to (189.5, 106.1), turned to 90 degrees
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Routing:
- net Net-(D50-A1): track 17.0 -> 56.1 mm
- net Net-(D60-A1): track 17.4 -> 56.2 mm
- net Net-(D70-A1): track 17.8 -> 56.2 mm
- net Net-(D80-A1): track 18.3 -> 56.3 mm
- net 5Vb: track 132.5 -> 163.2 mm
- net S80: track 54.7 -> 34.0 mm
- net S50: track 34.8 -> 14.4 mm
- net S60: track 32.9 -> 13.8 mm
- net S70: track 37.4 -> 23.8 mm
- net Net-(C82-Pad1): track 9.79 -> 6.26 mm
- net Net-(C72-Pad1): track 9.39 -> 6.07 mm
- net Net-(C52-Pad1): track 9.39 -> 6.25 mm
- net Net-(C62-Pad1): track 9.39 -> 6.25 mm
- net Net-(D40-A1): track 54.3 -> 56.3 mm
- net Net-(D30-A1): track 57.2 -> 56.2 mm
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Other:
- board text removed: "S5"
- board text removed: "S6"
- board text removed: "S7"
- board text removed: "S8"

Commit message: zf-filter r0.2
Routing:
- net GND: vias 224 -> 236
Other:
- board text added: "R1.0"
Changed lines of the file:
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@@
+		)
+	)
+	(gr_text "R1.0"
+		(at 210 85 0)
+		(layer "F.SilkS")
+		(effects
+			(font
+				(size 2 2)
+				(thickness 0.25)
+				(bold yes)
+			)
 		)
 	)
@@
 	)
 	(via
+		(at 192.5 87.5)
+		(size 0.6)
+		(drill 0.3)
+		(layers "F.Cu" "B.Cu")
+		(free yes)
+		(net 2)
+	)
+	(via
+		(at 122.5 82.5)
+		(size 0.6)
+		(drill 0.3)
+		(layers "F.Cu" "B.Cu")
+		(free yes)
+		(net 2)
+	)
+	(via
 		(at 137.5 117.5)
 		(size 0.6)
@@
 	)
 	(via
+		(at 192.5 82.5)
+		(size 0.6)
+		(drill 0.3)
+		(layers "F.Cu" "B.Cu")
+		(free yes)
+		(net 2)
+	)
+	(via
 		(at 212.5 85)
 		(size 0.6)
@@
 	)
 	(via
+		(at 120 87.5)
+		(size 0.6)
+		(drill 0.3)
+		(layers "F.Cu" "B.Cu")
+		(free yes)
+		(net 2)
+	)
+	(via
 		(at 120 110)
 		(size 0.6)
@@
 	)
 	(via
+		(at 122.5 87.5)
+		(size 0.6)
+		(drill 0.3)
+		(layers "F.Cu" "B.Cu")
+		(free yes)
+		(net 2)
+	)
+	(via
 		(at 92.5 120)
 		(size 0.6)
@@
 	)
 	(via
+		(at 117.5 82.5)
+		(size 0.6)
+		(drill 0.3)
+		(layers "F.Cu" "B.Cu")
+		(free yes)
+		(net 2)
+	)
+	(via
 		(at 125 92.5)
 		(size 0.6)
@@
 	)
 	(via
+		(at 187.5 82.5)
+		(size 0.6)
+		(drill 0.3)
+		(layers "F.Cu" "B.Cu")
+		(free yes)
+		(net 2)
+	)
+	(via
 		(at 95 117.5)
 		(size 0.6)
@@
 	)
 	(via
+		(at 120 82.5)
+		(size 0.6)
+		(drill 0.3)
+		(layers "F.Cu" "B.Cu")
+		(free yes)
+		(net 2)
+	)
+	(via
 		(at 190 120)
 		(size 0.6)
@@
 	)
 	(via
+		(at 117.5 87.5)
+		(size 0.6)
+		(drill 0.3)
+		(layers "F.Cu" "B.Cu")
+		(free yes)
+		(net 2)
+	)
+	(via
 		(at 210 117.5)
 		(size 0.6)
@@
 	)
 	(via
+		(at 190 82.5)
+		(size 0.6)
+		(drill 0.3)
+		(layers "F.Cu" "B.Cu")
+		(free yes)
+		(net 2)
+	)
+	(via
 		(at 107.5 112.5)
 		(size 0.6)
@@
 	)
 	(via
+		(at 187.5 87.5)
+		(size 0.6)
+		(drill 0.3)
+		(layers "F.Cu" "B.Cu")
+		(free yes)
+		(net 2)
+	)
+	(via
 		(at 140 87.5)
 		(size 0.6)
@@
 		(size 0.6)
 		(drill 0.3)
+		(layers "F.Cu" "B.Cu")
+		(free yes)
+		(net 2)
+	)
+	(via
+		(at 190 87.5)
+		(size 0.6)
+		(drill 0.3)
